File: Circuit/VX8Battery/VX8Battery.kicad_pcb (KiCad board)
At the start: 2 copper layers, 49 x 77.4 mm, 28 parts, among them J1 USBC-Molex-2171780001, J2 VX8BattPins, U1 MP2672A

Commit message: Mostly circuit board updates. Still need to fix the dependency chart for the case
Routing:
- net GND: track 189.5 -> 213.8 mm, vias 13 -> 16
- net Net-(BT1-Pad2): track 105.6 -> 114.1 mm
- net Net-(C3-Pad1): track 5.63 -> 5.09 mm
- added copper zone on B.Cu, net GND
- added copper zone on F.Cu, net GND
Other:
- board text added: "YAESU VX-8 Battery 21700 OR 18650 (With the right Keystone clips) 2021 AB1TJ"
